Commit message: update

File: install/share/arm/config/gazebo_kipps_arm.urdf (robot description, URDF)
Before this commit: robot kipps_arm, 7 links, 6 joints
Links:
- link base_link: geometry collision mesh filename=package://description/meshes/base_link.stl; visual mesh filename=package://description/meshes/base_link.stl
